Commit message: minor: Re-indent plane.urdf

File: upkie/cpp/actuation/bullet/plane/plane.urdf (robot description, URDF)
Before this commit: robot plane, 1 links, 0 joints
Links:
- removed link planeLink
- added link plane_link, mass .0; collision box size=200 200 10; visual mesh filename=plane.obj scale=1 1 1
